Commit message: i tried

File: simulation_ws/src/robot_description/urdf/robot.xacro (robot description, xacro)
@@ -1,79 +1,43 @@
 <?xml version="1.0" ?>
 <robot name="robot" xmlns:xacro="http://www.ros.org/wiki/xacro">
-  <material name="black">
-    <color rgba="0.0 0.0 0.0 1.0"/>
-  </material>
-  <material name="blue">
-    <color rgba="0.203125 0.23828125 0.28515625 1.0"/>
-  </material>
-  <material name="green">
-    <color rgba="0.0 0.8 0.0 1.0"/>
-  </material>
-  <material name="grey">
-    <color rgba="0.2 0.2 0.2 1.0"/>
-  </material>
-  <material name="orange">
-    <color rgba="1.0 0.423529411765 0.0392156862745 1.0"/>
-  </material>
-  <material name="brown">
-    <color rgba="0.870588235294 0.811764705882 0.764705882353 1.0"/>
-  </material>
-  <material name="red">
-    <color rgba="0.80078125 0.12890625 0.1328125 1.0"/>
-  </material>
-  <material name="white">
-    <color rgba="1.0 1.0 1.0 1.0"/>
-  </material>
-  <gazebo reference="link_chassis">
-    <material>Gazebo/Orange</material>
-  </gazebo>
-  <gazebo reference="link_left_wheel">
-    <material>Gazebo/Blue</material>
-  </gazebo>
-  <gazebo reference="link_right_wheel">
-    <material>Gazebo/Blue</material>
-  </gazebo>
-  <gazebo>
-    <plugin filename="libgazebo_ros_diff_drive.so" name="differential_drive_controller">
-      <legacyMode>false</legacyMode>
-      <alwaysOn>true</alwaysOn>
-      <updateRate>20</updateRate>
-      <leftJoint>joint_left_wheel</leftJoint>
-      <rightJoint>joint_right_wheel</rightJoint>
-      <wheelSeparation>0.2</wheelSeparation>
-      <wheelDiameter>0.2</wheelDiameter>
-      <torque>0.1</torque>
-      <commandTopic>cmd_vel</commandTopic>
-      <odometryTopic>odom</odometryTopic>
-      <odometryFrame>odom</odometryFrame>
-      <robotBaseFrame>link_chassis</robotBaseFrame>
-    </plugin>
-  </gazebo>
+  <xacro:property name="package_name" value="robot_description"/>
+  <xacro:property name="robot_name" value="robot"/>
+  <xacro:include filename="$(find ${package_name})/urdf/robot.gazebo"/>
+  <xacro:include filename="$(find ${package_name})/urdf/materials.xacro"/>
+  <xacro:include filename="$(find ${package_name})/urdf/macros.xacro"/>
+  <xacro:property name="base_length" value="0.5"/>
+  <xacro:property name="base_width" value="0.3"/>
+  <xacro:property name="base_height" value="0.07"/>
+  <xacro:property name="laser_sensor_size" value="0.05"/>
+  <xacro:property name="wheel_diam" value="0.2"/>
+  <xacro:property name="wheel_width" value="0.04"/>
+  <xacro:property name="collision_inflation" value="1.1"/>
+  <xacro:property name="wheel_x_pos" value="${base_length/4}"/>
+  <xacro:property name="wheel_y_pos" value="${base_width/2+wheel_width/2}"/>
+  <xacro:property name="wheel_z_pos" value="0"/>
+  <link name="base_footprint"/>
+  <joint name="joint_base_footprint" type="fixed">
+    <parent link="base_footprint"/>
+    <child link="link_chassis"/>
+    <origin xyz="0.0 0.0 ${wheel_diam/2}"/>
+  </joint>
   <link name="link_chassis">
-    <!-- pose and inertial -->
-    <pose>0 0 0.1 0 0 0</pose>
-    <inertial>
-      <mass value="5"/>
-      <origin rpy="0 0 0" xyz="0 0 0.1"/>
-      <inertia ixx="0.0395416666667" ixy="0" ixz="0" iyy="0.106208333333" iyz="0" izz="0.106208333333"/>
-    </inertial>
     <!-- body -->
     <collision name="collision_chassis">
       <geometry>
-        <box size="0.5 0.3 0.07"/>
+        <box size="${base_length*collision_inflation} ${base_width*collision_inflation} ${base_height*collision_inflation}"/>
       </geometry>
     </collision>
-    <visual>
-      <origin rpy="0 0 0" xyz="0 0 0"/>
+    <visual name="chassis_visual">
       <geometry>
-        <box size="0.5 0.3 0.07"/>
+        <box size="${base_length} ${base_width} ${base_height}"/>
       </geometry>
-      <material name="blue"/>
+      <material name="orange"/>
     </visual>
-    <!-- caster front -->
-    <collision name="caster_front_collision">
-      <origin rpy=" 0 0 0" xyz="0.35 0 -0.05"/>
+    <!-- caster -->
+    <collision name="caster_rear_collision">
+      <origin rpy=" 0 0 0" xyz="${-base_length/4} 0 ${-wheel_diam/4}"/>
       <geometry>
-        <sphere radius="0.05"/>
+        <sphere radius="${wheel_diam/4}"/>
       </geometry>
       <surface>
@@ -88,64 +52,55 @@
       </surface>
     </collision>
-    <visual name="caster_front_visual">
-      <origin rpy=" 0 0 0" xyz="0.2 0 -0.05"/>
+    <visual name="caster_rear_visual">
+      <origin rpy=" 0 0 0" xyz="${-base_length/4} 0 ${-wheel_diam/4}"/>
       <geometry>
-        <sphere radius="0.05"/>
+        <sphere radius="${wheel_diam/4}"/>
       </geometry>
+      <material name="blue"/>
     </visual>
+    <!-- pose and inertial -->
+    <pose>0 0 0.1 0 0 0</pose>
+    <xacro:base_inertia m="5" x="${base_length}" y="${base_width}" z="${base_height}"
+      o_xyz="0 0 0" o_rpy="0 0 0.1"/>
   </link>
-  <link name="link_right_wheel">
-    <inertial>
-      <mass value="0.2"/>
-      <origin rpy="0 1.5707 1.5707" xyz="0 0 0"/>
-      <inertia ixx="0.000526666666667" ixy="0" ixz="0" iyy="0.000526666666667" iyz="0" izz="0.001"/>
-    </inertial>
-    <collision name="link_right_wheel_collision">
-      <origin rpy="0 1.5707 1.5707" xyz="0 0 0"/>
+  <xacro:wheel side="right" base_link="link_chassis"
+    m="0.2" r="${wheel_diam/2}" l="${wheel_width}"
+    x_pos="${wheel_x_pos}" y_pos="${-wheel_y_pos}" z_pos="${wheel_z_pos}" />
+  <xacro:wheel side="left" base_link="link_chassis"
+    m="0.2" r="${wheel_diam/2}" l="${wheel_width}"
+    x_pos="${wheel_x_pos}" y_pos="${wheel_y_pos}" z_pos="${wheel_z_pos}" />
+  <joint name="joint_laser" type="fixed">
+    <axis xyz="0 1 0" />
+    <origin xyz="${base_length/2 + laser_sensor_size/2} 0 0" rpy="0 0 0"/>
+    <parent link="link_chassis"/>
+    <child link="link_laser"/>
+  </joint>
+  <!-- Hokuyo Laser -->
+  <link name="link_laser">
+    <collision>
+      <origin xyz="0 0 0" rpy="0 0 0"/>
       <geometry>
-        <cylinder length="0.04" radius="0.1"/>
+        <box size="${laser_sensor_size} ${laser_sensor_size} ${laser_sensor_size}"/>
       </geometry>
     </collision>
-    <visual name="link_right_wheel_visual">
-      <origin rpy="0 1.5707 1.5707" xyz="0 0 0"/>
+    <visual>
+      <origin xyz="${-laser_sensor_size/10} 0 0" rpy="0 0 0"/>
       <geometry>
-        <cylinder length="0.04" radius="0.1"/>
+        <box size="${laser_sensor_size*0.8} ${laser_sensor_size} ${laser_sensor_size}"/>
       </geometry>
+      <material name="green"/>
     </visual>
+    <visual>
+      <origin xyz="${laser_sensor_size*0.25} 0 0" rpy="0 0 0"/>
+      <geometry>
+        <box size="${laser_sensor_size*0.5} ${laser_sensor_size*0.5} ${laser_sensor_size*0.5}"/>
+      </geometry>
+      <material name="green"/>
+    </visual>
+    <inertial>
+      <mass value="1e-5" />
+      <origin xyz="0 0 0" rpy="0 0 0"/>
+      <inertia ixx="1e-6" ixy="0" ixz="0" iyy="1e-6" iyz="0" izz="1e-6" />
+    </inertial>
   </link>
-  <joint name="joint_right_wheel" type="continuous">
-    <origin rpy="0 0 0" xyz="-0.05 0.15 0"/>
-    <child link="link_right_wheel"/>
-    <parent link="link_chassis"/>
-    <axis rpy="0 0 0" xyz="0 1 0"/>
-    <limit effort="10000" velocity="1000"/>
-    <joint_properties damping="1.0" friction="1.0"/>
-  </joint>
-  <link name="link_left_wheel">
-    <inertial>
-      <mass value="0.2"/>
-      <origin rpy="0 1.5707 1.5707" xyz="0 0 0"/>
-      <inertia ixx="0.000526666666667" ixy="0" ixz="0" iyy="0.000526666666667" iyz="0" izz="0.001"/>
-    </inertial>
-    <collision name="link_left_wheel_collision">
-      <origin rpy="0 1.5707 1.5707" xyz="0 0 0"/>
-      <geometry>
-        <cylinder length="0.04" radius="0.1"/>
-      </geometry>
-    </collision>
-    <visual name="link_left_wheel_visual">
-      <origin rpy="0 1.5707 1.5707" xyz="0 0 0"/>
-      <geometry>
-        <cylinder length="0.04" radius="0.1"/>
-      </geometry>
-    </visual>
-  </link>
-  <joint name="joint_left_wheel" type="continuous">
-    <origin rpy="0 0 0" xyz="-0.05 -0.15 0"/>
-    <child link="link_left_wheel"/>
-    <parent link="link_chassis"/>
-    <axis rpy="0 0 0" xyz="0 1 0"/>
-    <limit effort="10000" velocity="1000"/>
-    <joint_properties damping="1.0" friction="1.0"/>
-  </joint>
 </robot>
